File: k2_v4.l4.kicad_pcb (KiCad board)
At the start: 6 copper layers, 120 x 46 mm, 42 parts, among them J11 J_EC_HEADER, J12 J_12V_IN, J13 J_SWD, J2 SlimSAS_x8_SFF8654, J3 MCIO_4i_SFF1016, J4 MCIO_4i_SFF1016, J6 J_PWR_CTRL, J9 J_OOB_HEADER, U1 STM32G0B1CBT6, U2 DCDC_12V_3V3, U4 BAT54C, U5 OPTO_LTV356T, U6 DS320PR1601

Commit message: feat(k2): ROOT-21 — 实施 O1b(REFCLK 差分对 P/N) + O3(L4 网名)；W3-CN.25 FEASIBLE_ALL；D8/G5 PASS；G7 仍 FAIL(O1/O2)
- W3 refclk_place 改为**差分对**：每页 P/N 两条路径，P/N 分离 >=0.38，成对中心取见证
  pair_centre_window_y/channel_y，keepout 零交（A-CN.5a PASS）；net 名取 manifest PCIE_REFCLK*_P/N
- W3 rev W3-CN.25：FEASIBLE_ALL（R1 32/32, same_layer 0, 全谓词 PASS, landing 重发射）
- L4 重发：68 网/338 段/256 via（REFCLK 4 段 × ...）；L4 validator PASS；dst board b63e6c09
- 验证器 v2：PASS（G-M3 per_copy 随公式修正；A1.3 V7 覆盖 REFCLK P/N）
- L5 重测：DFM 479（新增 N 轨 26 条）；SI skew 24.476 不变 => **G7 仍 FAIL**
- **O1 已实证不可行**（域 195916->571904 rows + 3 序均 R1 31/32）-> 需 owner（第4层/放宽净距/换架构）
- **O2 待裁决**（W3 零板读 -> 159 our<->frozen）；冻结四源 MATCH；零搜索
Routing:
- net PCIE_REFCLK1/input: track 87.4 -> 0.00 mm
- net PCIE_REFCLK1_N: track 0.00 -> 86.6 mm
- net PCIE_REFCLK1_P: track 0.00 -> 84.8 mm
- net PCIE_REFCLK0_N: track 0.00 -> 76.9 mm
- net PCIE_REFCLK0_P: track 0.00 -> 73.9 mm
- net PCIE_REFCLK0/input: track 73.8 -> 0.00 mm
