File: hw/sch/redriver_ds320pr1601_sideband_strap.kicad_sch (KiCad schematic)
At the start: 10 parts, among them U6 DS320PR1601

Commit message: p3(k2): #K2-16 §五 一次执行 —— 源侧 strap 0603 修复 + rev-24 逐端点 basis + L2 canonical 指引 + P3-3 55/55 + C7 口径 9 铜区
- 源侧：errata yaml 17d540f058631a5e 经 project.yaml:nets_yaml 生效；sch sheet c7099e2fae642bdd + 符号库 6b572ceb7ffc2e69（按源重出，其余 sheet 逐字节未变；冻结原件 dd794c54 未动）⇒ P3-3 = 55/55 实测、unresolved=[]
- rev-24 317140048c80a569：数值零变更（承 rev-23）+ 新增 corridors_clearance_basis_v24 逐端点留痕（65.05 实测 0 差 / 82.60,104.84 = L1 走廊模型 pad_extent_x 板实测 82.76,105.00 +0.16 / 132.65 = J2 slab 内缘 板实测 132.00 +0.65 混口径显式登记）+ project.yaml 重指向 + L3 README v5
- L2 canonical 指引：L2/README-canonical.md 1ad55180c4c74e65（8L canonical / 走廊口径 L2-4 / v2.0 6L 与 17.30-27.40 作废；不改 frozen 0444；含 In5/In6 待裁项）
- C7 口径修正 = 9 铜区（12V_IN×1/GND×3/MCU_VDD×1/P3V3×2/P3V3_AUX×2），4 个无网 ESC_* keepout 排除（#K2-16 §四 监理自纠）
- P3 图集 v8 50b14c183e603064；drawings 45b4a9ee4fdc4c4b；生成器 fa01d62895a4582d；图纸 README 12f109411a68e71e；P4 输入前置 v2 4e57c3ab35d6f568
- E1/E2/E3 复算未受扰动（板42/图55/网表55；板-图 0；489=424/15/50）；未动 criteria/冻结件；未派 WORKER
Parts:
- R35, R38: footprint R_0402_1005Metric -> Resistor_SMD:R_0603_1608Metric
- R36, R37, R39, R42, R43, R44, R45: footprint Resistor_SMD:R_0402_1005Metric -> Resistor_SMD:R_0603_1608Metric
Changed lines of the file:
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@@
       (property "Reference" "R35" (at 594.360 600.710 0) (hide no) (effects (font (size 1.27 1.27))) (id 0))
       (property "Value" "R_6K19" (at 594.360 588.010 0) (hide no) (effects (font (size 1.27 1.27))) (id 1))
-      (property "Footprint" "R_0402_1005Metric" (at 594.360 594.360 0) (hide yes) (effects (font (size 1.27 1.27))) (id 2))
+      (property "Footprint" "Resistor_SMD:R_0603_1608Metric" (at 594.360 594.360 0) (hide yes) (effects (font (size 1.27 1.27))) (id 2))
       (pin "1")
       (pin "2")
@@
       (property "Reference" "R36" (at 594.360 622.300 0) (hide no) (effects (font (size 1.27 1.27))) (id 0))
       (property "Value" "1K" (at 594.360 612.140 0) (hide no) (effects (font (size 1.27 1.27))) (id 1))
-      (property "Footprint" "Resistor_SMD:R_0402_1005Metric" (at 594.360 617.220 0) (hide yes) (effects (font (size 1.27 1.27))) (id 2))
+      (property "Footprint" "Resistor_SMD:R_0603_1608Metric" (at 594.360 617.220 0) (hide yes) (effects (font (size 1.27 1.27))) (id 2))
       (pin "1")
       (pin "2")
@@
       (property "Reference" "R37" (at 594.360 642.620 0) (hide no) (effects (font (size 1.27 1.27))) (id 0))
       (property "Value" "1K" (at 594.360 632.460 0) (hide no) (effects (font (size 1.27 1.27))) (id 1))
-      (property "Footprint" "Resistor_SMD:R_0402_1005Metric" (at 594.360 637.540 0) (hide yes) (effects (font (size 1.27 1.27))) (id 2))
+      (property "Footprint" "Resistor_SMD:R_0603_1608Metric" (at 594.360 637.540 0) (hide yes) (effects (font (size 1.27 1.27))) (id 2))
       (pin "1")
       (pin "2")
@@
       (property "Reference" "R38" (at 594.360 664.210 0) (hide no) (effects (font (size 1.27 1.27))) (id 0))
       (property "Value" "R_8K25" (at 594.360 651.510 0) (hide no) (effects (font (size 1.27 1.27))) (id 1))
-      (property "Footprint" "R_0402_1005Metric" (at 594.360 657.860 0) (hide yes) (effects (font (size 1.27 1.27))) (id 2))
+      (property "Footprint" "Resistor_SMD:R_0603_1608Metric" (at 594.360 657.860 0) (hide yes) (effects (font (size 1.27 1.27))) (id 2))
       (pin "1")
       (pin "2")
@@
       (property "Reference" "R39" (at 594.360 685.800 0) (hide no) (effects (font (size 1.27 1.27))) (id 0))
       (property "Value" "1K" (at 594.360 675.640 0) (hide no) (effects (font (size 1.27 1.27))) (id 1))
-      (property "Footprint" "Resistor_SMD:R_0402_1005Metric" (at 594.360 680.720 0) (hide yes) (effects (font (size 1.27 1.27))) (id 2))
+      (property "Footprint" "Resistor_SMD:R_0603_1608Metric" (at 594.360 680.720 0) (hide yes) (effects (font (size 1.27 1.27))) (id 2))
       (pin "1")
       (pin "2")
@@
       (property "Reference" "R42" (at 594.360 706.120 0) (hide no) (effects (font (size 1.27 1.27))) (id 0))
       (property "Value" "1K" (at 594.360 695.960 0) (hide no) (effects (font (size 1.27 1.27))) (id 1))
-      (property "Footprint" "Resistor_SMD:R_0402_1005Metric" (at 594.360 701.040 0) (hide yes) (effects (font (size 1.27 1.27))) (id 2))
+      (property "Footprint" "Resistor_SMD:R_0603_1608Metric" (at 594.360 701.040 0) (hide yes) (effects (font (size 1.27 1.27))) (id 2))
       (pin "1")
       (pin "2")
@@
       (property "Reference" "R43" (at 594.360 726.440 0) (hide no) (effects (font (size 1.27 1.27))) (id 0))
       (property "Value" "1K" (at 594.360 716.280 0) (hide no) (effects (font (size 1.27 1.27))) (id 1))
-      (property "Footprint" "Resistor_SMD:R_0402_1005Metric" (at 594.360 721.360 0) (hide yes) (effects (font (size 1.27 1.27))) (id 2))
+      (property "Footprint" "Resistor_SMD:R_0603_1608Metric" (at 594.360 721.360 0) (hide yes) (effects (font (size 1.27 1.27))) (id 2))
       (pin "1")
       (pin "2")
@@
       (property "Reference" "R44" (at 594.360 746.760 0) (hide no) (effects (font (size 1.27 1.27))) (id 0))
       (property "Value" "1K" (at 594.360 736.600 0) (hide no) (effects (font (size 1.27 1.27))) (id 1))
-      (property "Footprint" "Resistor_SMD:R_0402_1005Metric" (at 594.360 741.680 0) (hide yes) (effects (font (size 1.27 1.27))) (id 2))
+      (property "Footprint" "Resistor_SMD:R_0603_1608Metric" (at 594.360 741.680 0) (hide yes) (effects (font (size 1.27 1.27))) (id 2))
       (pin "1")
       (pin "2")
@@
       (property "Reference" "R45" (at 594.360 767.080 0) (hide no) (effects (font (size 1.27 1.27))) (id 0))
       (property "Value" "1K" (at 594.360 756.920 0) (hide no) (effects (font (size 1.27 1.27))) (id 1))
-      (property "Footprint" "Resistor_SMD:R_0402_1005Metric" (at 594.360 762.000 0) (hide yes) (effects (font (size 1.27 1.27))) (id 2))
+      (property "Footprint" "Resistor_SMD:R_0603_1608Metric" (at 594.360 762.000 0) (hide yes) (effects (font (size 1.27 1.27))) (id 2))
       (pin "1")
       (pin "2")
