File: hw/sch/mcu_sideband.kicad_sch (KiCad schematic)
At the start: 21 parts, among them J11 J_EC_HEADER, J13 J_OOB_HEADER, J6 J_PWR_CTRL, J9 J_OOB_HEADER, U1 STM32G0B1CBT6, U5 OPTO_LTV356T

Commit message: fix(K2/#K2-57 R1+R2+R3+R4+R5+R6): CR-26 U4 BAT54C ORing 反接修复链落地 (新 rev 前置) + CR-27 并入 + 引证 5 项 + CR-32/CR-33 在册
R1(真源·四树): BAT54C.yaml 1:A1/2:A2/3:K (另笔于 _shared 四树)
R3(新 rev 前置·网表): 新增 hw/data/k2_sch.errata-3.yaml -- 仅订正 pin NAME->NUMBER
  BAT54C_ORING K 2->3 / A2 3->2 ; LED A 1->2 / K 2->1
  nets 逐字不动(100); k2_sch.yaml 逐字节未改 (dd794c54f7ce7417 => 判据 ④)
  pm_gate/project.yaml + pipeline.yaml nets_yaml -> errata-3 (版本 bump, 同 owner #K2-24 先例)
R2(符号层·有效杠杆澄清): IOCONVERT.kicad_sym#BAT54C_ORING -> K=3/A2=2;
  内嵌 sch (power_12v_...) 同步; 见 CR-33
R4(CR-27 并入): IOCONVERT.kicad_sym#LED -> A=2/K=1 + mcu_sideband.kicad_sch 同步
  (前置: 本机官方 LED_0603_1608Metric pad1 左侧 x=-0.7875, 阴极丝印 x=-1.485 => pad1=K)
R5(引证): 见 _shared 四树笔
R6(过程口径): CR-32 在册 (待裁项须结构化, 禁只写 handoff/ledger)

复算证据 (k2_gen_v5 双跑对照):
  errata-2: U4 pad2=MCU_VDD / pad3=P3V3   (复现缺陷)
  errata-3: U4 pad2=P3V3   / pad3=MCU_VDD (实体 A2->P3V3, K->MCU_VDD => 正向导通) OK
            D1 pad1=GND    / pad2=LED_A   (正向) OK
gate: sch_structural/netlist_connect/bom_consistent/project_sch_coverage 全 PASS
Connections:
- net GND: now also D1.1 (K); no longer D1.2 (K)
- net LED_A: now also D1.2 (A); no longer D1.1 (A)
